File: roPlug.kicad_pcb (KiCad board)
At the start: 2 copper layers, 25 x 26 mm, 18 parts, among them P1 USB_C_Plug, SW1 Rotary_Encoder_Switch, U1 ATmega32U4-MU, Y1 16MHz

Commit message: add more connection to ground
Routing:
- net GND: track 49.1 -> 50.8 mm
